File: edge/co2sensor/hardware/lp8-module.kicad_pcb (KiCad board)
At the start: 2 copper layers, 28 parts, among them J1 Conn_01x05_Male, J2 Conn_01x06_Male, J3 Conn_01x01_Male, J4 Conn_01x01_Male, Q1 PMOS-SI2315BDS-T1-E3, Q2 PMOS-SI2315BDS-T1-E3, Q3 PMOS-SI2315BDS-T1-E3, U1 MAX6006/LT1634, U2 MCP6041T-EOT, U3 TPS22917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

Commit message: latest fab files
Parts:
- Q3, R11, R12, R9, U4: moved to F.Cu
- moved U4 18.0 mm to (158.9, 103.8), turned to 0 degrees
- moved R9 15.3 mm to (156.3, 105.1), turned to 90 degrees
- moved C3 2.54 mm to (159.0, 101.3)
- moved Q3 1.02 mm to (144.9, 88.8), turned to 0 degrees
Connections:
- C3 pad 1: /LP8_VCAP -> Net-(C3-Pad1)
- Q1 pad 3: Net-(Q1-Pad3) -> /LP8_VCAP
- Q2 pad 2: /LP8_VCAP -> Net-(C3-Pad1)
- Q2 pad 3: Net-(Q1-Pad3) -> /LP8_VCAP
- R7 pad 1: /LP8_VCAP -> Net-(C3-Pad1)
- U4 pad 1: /LP8_VCAP -> Net-(C3-Pad1)
Routing:
- net /LP8_VCAP: track 59.5 -> 24.9 mm, vias 2 -> 1
- net Net-(A1-Pad1.1): track 6.89 -> 24.5 mm
- net Net-(C3-Pad1): track 0.00 -> 15.3 mm, vias 0 -> 2
- net GND: track 127.2 -> 118.1 mm
- net /LP8_EN_MEAS: track 49.0 -> 42.9 mm, vias 1 -> 2
- net /LP8/LP8_3V3: track 101.0 -> 105.6 mm
- net /LP8/V+: track 14.3 -> 12.7 mm
- net /RxD: track 18.0 -> 16.5 mm
- net Net-(Q3-Pad1): track 4.93 -> 6.33 mm
- net /TxD: track 23.1 -> 22.0 mm
- net /LP8_MEAS_RDY: track 11.4 -> 11.9 mm
